Commit message: added unified launch file

File: qubo_sim/urdf/gazebo.xacro (robot description, xacro)
@@ -2,5 +2,5 @@
 <robot xmlns:xacro="http://www.ros.org/wiki/xacro">
     <!-- Center of buoyancy -->
-    <xacro:property name="qubo_gazebo_cob" value="0 0 0.04"/>
+    <xacro:property name="qubo_gazebo_cob" value="0 0.22 0.2"/>
     <!-- Vehicle's actual volume (Gazebo cannot compute the volume out of the mesh) -->
     <xacro:property name="qubo_gazebo_volume" value="1"/>
