Commit message: nbrfQubo.launch can find all meshes now. Need to export launches correctly so they're available from anywhere after a catkin_make and source devel/setup.bash

File: qubo_sim/qubo_config.xacro (robot description, xacro)
@@ -4,6 +4,6 @@
   <xacro:arg name="namespace" default="qubo_gazebo"/>
   <!-- Include the ROV macro file -->
-  <xacro:include filename="$(find qubo_gazebo_description)/urdf/base.xacro"/>
-  <xacro:include filename="$(find qubo_gazebo_description)/urdf/gazebo.xacro"/>
+  <xacro:include filename="$(find qubo-gazebo)/qubo_sim/urdf/base.xacro"/>
+  <xacro:include filename="$(find qubo-gazebo)/qubo_sim/urdf/gazebo.xacro"/>
   <!-- Create the qubo_gazebo -->
   <xacro:qubo_gazebo_base namespace="$(arg namespace)">

File: qubo_sim/urdf/base.xacro (robot description, xacro)
@@ -8,6 +8,6 @@
   <xacro:include filename="$(find uuv_gazebo_ros_plugins)/urdf/snippets.xacro"/>
   <!-- Loading vehicle's specific macros -->
-  <xacro:include filename="$(find qubo_gazebo_description)/urdf/snippets.xacro"/>
-  <xacro:include filename="$(find qubo_gazebo_description)/urdf/materials.xacro" />
+  <xacro:include filename="$(find qubo-gazebo)/qubo_sim/urdf/snippets.xacro"/>
+  <xacro:include filename="$(find qubo-gazebo)/qubo_sim/urdf/materials.xacro" />
   <!--
     Vehicle's parameters (remember to enter the model parameters below)
@@ -24,9 +24,9 @@
     Open the meshes for the RexROV vehicle in Blender to see an example on the mesh placement.
   -->
-  <xacro:property name="visual_mesh_file" value="file://$(find qubo_gazebo_description)/meshes/vehicle.stl"/>
+  <xacro:property name="visual_mesh_file" value="file://$(find qubo-gazebo)/qubo_sim/meshes/vehicle.stl"/>
   <!-- Collision geometry mesh, usually in STL format (it is recommended to keep
   this geometry as simple as possible to improve the performance the physics engine
   regarding the computation of collision forces) -->
-  <xacro:property name="collision_mesh_file" value="file://$(find qubo_gazebo_description)/meshes/vehicle.stl"/>
+  <xacro:property name="collision_mesh_file" value="file://$(find qubo-gazebo)/qubo_sim/meshes/vehicle.stl"/>
   <!-- Vehicle macro -->
   <xacro:macro name="qubo_gazebo_base" params="namespace *gazebo">
@@ -62,7 +62,7 @@
     <xacro:insert_block name="gazebo"/>
     <!-- Include the thruster modules -->
-    <xacro:include filename="$(find qubo_gazebo_description)/urdf/actuators.xacro"/>
+    <xacro:include filename="$(find qubo-gazebo)/qubo_sim/urdf/actuators.xacro"/>
     <!-- Include the sensor modules -->
-    <xacro:include filename="$(find qubo_gazebo_description)/urdf/sensors.xacro"/>
+    <xacro:include filename="$(find qubo-gazebo)/qubo_sim/urdf/sensors.xacro"/>
   </xacro:macro>
 </robot>

File: qubo_sim/urdf/snippets.xacro (robot description, xacro)
@@ -7,5 +7,5 @@
   over propeller's frame X-axis in DAE (Collada) or STL format.
   -->
-  <xacro:property name="prop_mesh_file" value="file://$(find qubo_gazebo_description)/meshes/propeller.dae"/>
+  <xacro:property name="prop_mesh_file" value="file://$(find qubo-gazebo)/qubo_sim/meshes/propeller.dae"/>
   <!--
     Thruster macro with integration of joint and link. The thrusters should
@@ -106,5 +106,5 @@
   -->
   <!-- A separate mesh for the fin should be stored in the meshes folder -->
-  <xacro:property name="fin_mesh_file" value="file://$(find qubo_gazebo_description)/meshes/fin.dae"/>
+  <xacro:property name="fin_mesh_file" value="file://$(find qubo-gazebo)/qubo_sim/meshes/fin.dae"/>
   <!-- Fin joint limits  -->
   <xacro:property name="fin_min_joint_limit" value="${0.0 * d2r}"/>

Commit message: made simulation nicer

File: qubo_sim/qubo_config.xacro (robot description, xacro)
@@ -1,31 +1,227 @@
 <?xml version="1.0"?>
-<robot name="qubo_gazebo" xmlns:xacro="http://www.ros.org/wiki/xacro" >
-  <xacro:arg name="debug" default="0"/>
-  <xacro:arg name="namespace" default="qubo_gazebo"/>
-  <!-- Include the ROV macro file -->
-  <xacro:include filename="$(find qubo-gazebo)/qubo_sim/urdf/base.xacro"/>
-  <xacro:include filename="$(find qubo-gazebo)/qubo_sim/urdf/gazebo.xacro"/>
-  <!-- Create the qubo_gazebo -->
-  <xacro:qubo_gazebo_base namespace="$(arg namespace)">
-    <!-- The underwater object plugin is given as an input block parameter to
-     allow the addition of external models of manipulator units -->
+<robot name="gazebo_qubo" xmlns:xacro="http://www.ros.org/wiki/xacro" >
+  <!-- Includes -->
+  <xacro:include filename="$(find uuv_descriptions)/urdf/common.urdf.xacro"/>
+  <xacro:include filename="$(find uuv_sensor_ros_plugins)/urdf/sensor_snippets.xacro"/>
+  <!-- Parameters -->
+  <xacro:property name="debug" value="0"/>
+  <!-- don't be fooled, if you want to change qubo's namespace, change the parameter below , and the name parameter above -->
+  <xacro:property name="namespace" value="gazebo_qubo"/>
+  <xacro:property name="prop_mesh_file" value="file://$(find qubo-gazebo)/qubo_sim/meshes/propeller.dae"/>
+  <xacro:property name="visual_mesh_file" value="file://$(find qubo-gazebo)/qubo_sim/meshes/vehicle.dae"/>
+  <xacro:property name="collision_mesh_file" value="file://$(find qubo-gazebo)/qubo_sim/meshes/vehicle.stl"/>
+  <!-- Qubo's mass, volume, and center of buoyancy -->
+  <xacro:property name="mass" value="21.5"/>
+  <xacro:property name="volume" value="0.0213186821"/>
+  <xacro:property name="center_of_buoyancy" value="0.0 0.0 0.2"/>
+  <!-- size of robot to meters X = .4064Z  Y = Z = .3048 -->
+  <!-- Qubo's base link. Assume a right-handed coordinate system, with x forward and z up -->
+  <link name="${namespace}/base_link">
+    <visual>
+      <geometry>
+        <mesh filename="${visual_mesh_file}" scale=".01 .01 .01" />
+      </geometry>
+      <origin xyz="0 0 0" rpy="0 0 3.14159265"/>
+    </visual>
+    <collision>
+      <geometry>
+        <mesh filename="${collision_mesh_file}" scale=".01 .01 .01" />
+      </geometry>
+      <origin xyz="0 0 0" rpy="1.5707963 0 3.14159265"/>
+    </collision>
+    <inertial>
+      <mass value="${mass}"/>
+      <origin xyz="0 0 0"/>
+      <inertia ixx="0.297155" ixy="0.0026542" ixz="0.0079437" iyy="0.435426" iyz="0.003223" izz="0.570213"/>
+    </inertial>
+  </link>
+  <!-- TODO: figure out what this does -->
+  <xacro:dummy_link name="${namespace}/ned_link" />
+  <joint name="ned_joint" type="fixed">
+    <!-- This is revolute and not static since gazebo would remove ned_link -->
+    <origin xyz="0 0 0" rpy="${pi} 0 0"/>
+    <parent link="${namespace}/base_link"/>
+    <child link="${namespace}/ned_link"/>
+    <limit effort="0" lower="0" upper="0" velocity="0"/>
+  </joint>
+  <!-- Set up hydrodynamic plugin  -->
+  <gazebo>
+    <plugin name="uuv_plugin" filename="libuuv_underwater_object_ros_plugin.so">
+      <fluid_density>1024.0</fluid_density>
+      <flow_velocity_topic>hydrodynamics/current_velocity</flow_velocity_topic>
+      <debug>${debug}</debug>
+      <link name="${namespace}/base_link">
+        <neutrally_buoyant>0</neutrally_buoyant>
+        <volume>${volume}</volume>
+        <box>
+          <width>.5334</width>
+          <length>.61565</length>
+          <height>.492125</height>
+        </box>
+        <center_of_buoyancy>${center_of_buoyancy}</center_of_buoyancy>
+        <!-- Added mass: see p.28 in Berg2012 -->
+        <!-- sgillen@20170205-13:02 - literally just scaled all these by a factor of 100 -->
+        <hydrodynamic_model>
+          <type>fossen</type>
+          <added_mass>
+             7.7979 -0.068773 -1.0332 .085426 -1.6554 -.078033
+            -.068773 12.22 0.5129 4.0944 -0.058488 0.62726
+              -1.0332 0.5129 36.599 0.61112 -3.8642 0.10774
+              .085426 4.0944 .061112 5.349 -0.10027 0.21019
+              -1.6554 -.058488 -3.8642 -0.10027 8.4269 -.011162
+              -.078033 0.62726 0.10775 0.21019 -.011162 2.2432
+          </added_mass>
+           <!-- Linear damping: see p.31 in Berg2012 -->
+          <linear_damping>-1.4 -1.3 -1.4 -5 -6 -2</linear_damping>
+          <!-- Non-linear damping: see p.30 in Berg2012 -->
+          <quadratic_damping>-15 -20 -36 -13 -15 -10</quadratic_damping>
+        </hydrodynamic_model>
+      </link>
+    </plugin>
+  </gazebo>
+  <!-- thrusters -->
+  <!-- ============================================================================== -->
+  <!-- Thruster joint and link macro -->
+  <xacro:macro name="thruster_macro" params="namespace thruster_id *origin">
+    <joint name="${namespace}/thruster_${thruster_id}_joint" type="continuous">
+      <xacro:insert_block name="origin"/>
+      <axis xyz="1 0 0"/>
+      <parent link="${namespace}/base_link"/>
+      <child link="${namespace}/thruster_${thruster_id}"/>
+    </joint>
+    <link name="${namespace}/thruster_${thruster_id}">
+      <xacro:box_inertial x="0" y="0" z="0" mass="0.01">
+        <origin xyz="0 0 0" rpy="0 0 0"/>
+      </xacro:box_inertial>
+      <visual>
+        <origin rpy="0 0 0" xyz="0 0 0"/>
+        <geometry>
+          <mesh filename="${prop_mesh_file}" scale=".4 .4 .4"/>
+        </geometry>
+      </visual>
+      <collision>
+        <origin xyz="0 0 0" rpy="0 ${0.5*pi} 0"/>
+        <geometry>
+          <cylinder length="0.000001" radius="0.000001"/>
+        </geometry>
+      </collision>
+    </link>
     <gazebo>
-      <plugin name="uuv_plugin" filename="libuuv_underwater_object_ros_plugin.so">
-        <fluid_density>1028.0</fluid_density>
-        <flow_velocity_topic>hydrodynamics/current_velocity</flow_velocity_topic>
-        <debug>$(arg debug)</debug>
-        <!-- Adding the hydrodynamic and hydrostatic parameters for the vehicle-->
-        <xacro:qubo_gazebo_hydro_model namespace="$(arg namespace)"/>
-        <!--
-          In case other modules are added to the vehicle (such as a manipulator)
-          that also have link running with the underwater object plugin, they
-          should also be added in this block. For this, this new module should
-          have a file similar to gazebo.xacro above with the description of the
-          parameter necessary for the underwater object plugin to be initialized.
-        -->
+      <plugin name="${namespace}_${thruster_id}_thruster_model" filename="libuuv_thruster_ros_plugin.so">
+        <linkName>${namespace}/thruster_${thruster_id}</linkName>
+        <jointName>${namespace}/thruster_${thruster_id}_joint</jointName>
+        <thrustTopic>${namespace}/thrusters/${thruster_id}/thrust</thrustTopic>
+        <inputTopic>${namespace}/thrusters/${thruster_id}/input</inputTopic>
+        <thrusterID>${thruster_id}</thrusterID>
+        <dynamics>
+          <type>FirstOrder</type>
+          <timeConstant>0.05</timeConstant>
+        </dynamics>
+        <conversion>
+          <type>Basic</type>
+          <rotorConstant>.05</rotorConstant>
+        </conversion>
       </plugin>
     </gazebo>
-  </xacro:qubo_gazebo_base>
-  <!-- Joint state publisher plugin -->
-  <xacro:default_joint_state_publisher namespace="$(arg namespace)" update_rate="10"/>
+  </xacro:macro>
+  <!-- yaw thrusters - Z = 5 inches from bottom, X = 9.28 inches from center, Y = 7.87 inches from center -->
+  <!-- Z = .127 X = .23 Y = .1998 -->
+  <!-- Attach thrusters to base link using macro defined above -->
+  <!-- thruster configs found here https://docs.google.com/presentation/d/1mApi5nQUcGGsAsevM-5AlKPS6-FG0kfG9tn8nH2BauY/edit#slide=id.g1d529f9e65_0_3 -->
+  <xacro:thruster_macro namespace="${namespace}" thruster_id="0">
+      <origin xyz="0.2 0.44 0.165" rpy="0 0 ${-pi/4}" />
+  </xacro:thruster_macro>
+  <xacro:thruster_macro namespace="${namespace}" thruster_id="1">
+      <origin xyz="0.2 -0.03 0.165" rpy="0 0 ${pi/4}" />
+  </xacro:thruster_macro>
+  <xacro:thruster_macro namespace="${namespace}" thruster_id="2">
+    <origin xyz="-0.2 -0.03 0.165" rpy="0 0 ${3*pi/4}" />
+  </xacro:thruster_macro>
+  <xacro:thruster_macro namespace="${namespace}" thruster_id="3">
+    <origin xyz="-0.2 0.44 0.165" rpy="0 0 ${-3*pi/4}" />
+  </xacro:thruster_macro>
+  <xacro:thruster_macro namespace="${namespace}" thruster_id="4">
+    <origin xyz="0.105 0.455 0.08" rpy="0 ${pi/2} 0" />
+  </xacro:thruster_macro>
+  <xacro:thruster_macro namespace="${namespace}" thruster_id="5">
+    <origin xyz="0.105 -0.05 0.08" rpy="0 ${pi/2} 0" />
+  </xacro:thruster_macro>
+  <xacro:thruster_macro namespace="${namespace}" thruster_id="6">
+    <origin xyz="-0.105 -0.05 0.08" rpy="0 ${pi/2} 0" />
+  </xacro:thruster_macro>
+  <xacro:thruster_macro namespace="${namespace}" thruster_id="7">
+    <origin xyz="-0.105 0.455 0.08" rpy="0 ${pi/2} 0" />
+  </xacro:thruster_macro>
+  <!-- sensors -->
+  <!-- ============================================================================== -->
+  <!-- Mount a 3D pose sensor -->
+  <link name="${namespace}/pose_sensor_link">
+    <xacro:box_inertial x="0" y="0" z="0" mass="0.01">
+      <origin xyz="0 0 0" rpy="0 0 0"/>
+    </xacro:box_inertial>
+    <visual>
+      <geometry>
+        <box size="0.1 0.1 0.1"/>
+      </geometry>
+    </visual>
+    <xacro:no_collision/>
+  </link>
+  <joint name="${namespace}/pose_sensor_joint" type="revolute">
+    <origin xyz="0 0 0" rpy="0 0 0"/>
+    <axis xyz="0 0 1"/>
+    <parent link="${namespace}/base_link"/>
+    <child link="${namespace}/pose_sensor_link"/>
+    <limit effort="0" lower="0" upper="0" velocity="0"/>
+  </joint>
+  <!-- Mount a 3D pose sensor -->
+  <link name="${namespace}/pressure_link">
+    <xacro:box_inertial x="0" y="0" z="0" mass="0.01">
+      <origin xyz="0 0 0" rpy="0 0 0"/>
+    </xacro:box_inertial>
+    <visual>
+      <geometry>
+        <box size="0.1 0.1 0.1"/>
+      </geometry>
+    </visual>
+    <xacro:no_collision/>
+  </link>
+  <!-- joint for pressure sensor, you need a joint to modify the parameters, if you just use the default xacro macro it makes a joint for you -->
+  <joint name="${namespace}/pressure_joint" type="revolute">
+    <origin xyz="0 0 0" rpy="0 0 0"/>
+    <axis xyz="0 0 1"/>
+    <parent link="${namespace}/base_link"/>
+    <child link="${namespace}/pressure_link"/>
+    <limit effort="0" lower="0" upper="0" velocity="0"/>
+  </joint>
+  <gazebo>
+    <plugin name="pose_3d_plugin" filename="libgazebo_ros_p3d.so">
+      <robotNamespace>${namespace}</robotNamespace>
+      <bodyName>${namespace}/base_link</bodyName>
+      <topicName>pose_gt</topicName>
+      <frameName>world</frameName>
+      <gaussianNoise>0.0349</gaussianNoise> <!-- our noise from the AHRS is 2 degrees rms -->
+      <updateRate>30</updateRate>
+    </plugin>
+  </gazebo>
+  <!-- DVL -->
+  <!-- <xacro:default_dvl namespace="${namespace}" parent_link="${namespace}/base_link"> -->
+  <!--   <origin xyz="-1.4 0 -0.312" rpy="0 ${0.5*pi} 0"/> -->
+  <!-- </xacro:default_dvl> -->
+  <!-- Pressure  -->
+  <!-- <xacro:default_pressure namespace="${namespace}" parent_link="${namespace}/base_link"> -->
+  <!--   <origin xyz="0 0 0" rpy="0 0 0"/> -->
+  <!--   <stddev>.01</stddev> -->
+  <!-- </xacro:default_pressure> -->
+  <!-- these should match the bar 30 on qubo, up to 300 kpa , with an absolute error absolute error of 5 kpa I assumed absolute error is about 3 * stddevs giving std dev of   -->
+  <!-- IMU  -->
+  <xacro:default_imu namespace="${namespace}" parent_link="${namespace}/base_link">
+    <origin xyz="0 0 0" rpy="0 0 0"/>
+  </xacro:default_imu>
+  <!-- Camera -->
+  <!-- the camera used the robot name + given namespace as it's namespace, so we omit the latter since the robot name is our namespace -->
+  <xacro:default_camera namespace="${namespace}" parent_link="${namespace}/base_link" suffix="cam1">
+    <origin xyz="0 .49 0.2" rpy="0 0 1.57079632679"/>
+  </xacro:default_camera>
+  <!-- Joint state publisher -->
+<!--  <xacro:default_joint_state_publisher namespace="qubo_test" update_rate="500"/> -->
 </robot>
